Commit message: waybo_base with lbr_iisy11

File: kuka_lbr_iisy_support/urdf/lbr_iisy11_r1300.urdf.xacro (robot description, xacro)
@@ -1,7 +1,254 @@
-<?xml version="1.0"?>
+<?xml version="1.0" encoding="UTF-8"?>
 <robot xmlns:xacro="http://www.ros.org/wiki/xacro" name="lbr_iisy11_r1300">
-  <!-- Import iisy urdf file  -->
+  <!-- include helper xacros -->
+  <xacro:include filename="$(find kuka_lbr_iisy_support)/urdf/lbr_iisy_ros2_control.xacro"/>
+  <xacro:include filename="$(find kuka_resources)/urdf/common_materials.xacro"/>
+  <xacro:include filename="$(find kuka_lbr_iisy_support)/urdf/lbr_iisy_transmission.xacro"/>
+  <!-- Define prefix argument -->
+  <xacro:arg name="prefix" default=""/>
+  <xacro:arg name="controller_ip" default="0.0.0.0"/>
+  <xacro:arg name="client_ip" default="0.0.0.0"/>
+  <xacro:arg name="use_fake_hardware" default="false"/>
+  <xacro:arg name="roundtrip_time" default="0"/>
+  <xacro:arg name="qos_config_file" default=""/>
+  <xacro:arg name="x" default="0"/>
+  <xacro:arg name="y" default="0"/>
+  <xacro:arg name="z" default="0"/>
+  <xacro:arg name="roll" default="0"/>
+  <xacro:arg name="pitch" default="0"/>
+  <xacro:arg name="yaw" default="0"/>
+  <xacro:macro name="kuka_lbr_iisy11_r1300_robot" params="prefix controller_ip client_ip use_fake_hardware roundtrip_time qos_config_file *origin">
+    <!-- ros2 control instance -->
+    <xacro:kuka_lbr_iisy_ros2_control name="${prefix}lbr_iisy11_r1300" prefix="${prefix}" client_ip="${client_ip}" controller_ip="${controller_ip}" use_fake_hardware="${use_fake_hardware}" roundtrip_time="${roundtrip_time}" qos_config_file="${qos_config_file}"/>
+    <!-- links - main serial chain -->
+    <link name="world"/>
+    <link name="waybo_base">
+      <collision>
+        <geometry>
+          <mesh filename="package://kuka_lbr_iisy_support/meshes/waybo_base/collision/waybo_base.STL"/>
+        </geometry>
+      </collision>
+      <visual>
+        <geometry>
+          <mesh filename="package://kuka_lbr_iisy_support/meshes/waybo_base/visual/waybo_base.STL"/>
+        </geometry>
+      </visual>
+    </link>
+    <link name="${prefix}base_link">
+      <collision>
+        <geometry>
+          <mesh filename="package://kuka_lbr_iisy_support/meshes/lbr_iisy11_r1300/collision/base_link.stl"/>
+        </geometry>
+        <origin rpy="0 0 0" xyz="0 0 0"/>
+      </collision>
+      <visual>
+        <geometry>
+          <mesh filename="package://kuka_lbr_iisy_support/meshes/lbr_iisy11_r1300/visual/base_link.stl"/>
+        </geometry>
+        <origin rpy="0 0 0" xyz="0 0 0"/>
+        <xacro:material_kuka_ral_pure_white/>
+      </visual>
+    </link>
+    <link name="${prefix}link_1">
+      <collision>
+        <geometry>
+          <mesh filename="package://kuka_lbr_iisy_support/meshes/lbr_iisy11_r1300/collision/link_1.stl"/>
+        </geometry>
+        <origin rpy="0 0 0" xyz="0 0 0"/>
+      </collision>
+      <inertial>
+        <inertia ixx="0.0489108039022503" ixy="0.0" ixz="0.0" iyy="0.038370593540088" iyz="0.0" izz="0.0522121642769911"/>
+        <mass value="9.62"/>
+        <origin rpy="-1.3035636348359196 -0.7815781053554712 1.2529437882898178" xyz="0.00344301039501039 0.0191980353430353 -0.08662803846153849"/>
+      </inertial>
+      <visual>
+        <geometry>
+          <mesh filename="package://kuka_lbr_iisy_support/meshes/lbr_iisy11_r1300/visual/link_1.stl"/>
+        </geometry>
+        <origin rpy="0 0 0" xyz="0 0 0"/>
+        <xacro:material_kuka_ral_pure_white/>
+      </visual>
+    </link>
+    <link name="${prefix}link_2">
+      <collision>
+        <geometry>
+          <mesh filename="package://kuka_lbr_iisy_support/meshes/lbr_iisy11_r1300/collision/link_2.stl"/>
+        </geometry>
+        <origin rpy="0 0 0" xyz="0 0 0"/>
+      </collision>
+      <inertial>
+        <inertia ixx="0.609923712050298" ixy="0.0" ixz="0.0" iyy="0.0385097671170806" iyz="0.0" izz="0.617803845441985"/>
+        <mass value="9.86515786038357"/>
+        <origin rpy="-0.0037282594736534596 -0.018939981545576166 -1.569953728930981" xyz="0.249085185084359 -0.00442629366790902 -0.0535128397562821"/>
+      </inertial>
+      <visual>
+        <geometry>
+          <mesh filename="package://kuka_lbr_iisy_support/meshes/lbr_iisy11_r1300/visual/link_2.stl"/>
+        </geometry>
+        <origin rpy="0 0 0" xyz="0 0 0"/>
+        <xacro:material_kuka_ral_pure_white/>
+      </visual>
+    </link>
+    <link name="${prefix}link_3">
+      <collision>
+        <geometry>
+          <mesh filename="package://kuka_lbr_iisy_support/meshes/lbr_iisy11_r1300/collision/link_3.stl"/>
+        </geometry>
+        <origin rpy="0 0 0" xyz="0 0 0"/>
+      </collision>
+      <inertial>
+        <inertia ixx="0.0181557035426496" ixy="0.0" ixz="0.0" iyy="0.0346916391676837" iyz="0.0" izz="0.037776951242458"/>
+        <mass value="7.49283573690527"/>
+        <origin rpy="0.1692981167548117 0.5271433699021747 -2.9605806714357508" xyz="0.0438696763639649 -0.00482189531013714 0.044913251068375"/>
+      </inertial>
+      <visual>
+        <geometry>
+          <mesh filename="package://kuka_lbr_iisy_support/meshes/lbr_iisy11_r1300/visual/link_3.stl"/>
+        </geometry>
+        <origin rpy="0 0 0" xyz="0 0 0"/>
+        <xacro:material_kuka_ral_pure_white/>
+      </visual>
+    </link>
+    <link name="${prefix}link_4">
+      <collision>
+        <geometry>
+          <mesh filename="package://kuka_lbr_iisy_support/meshes/lbr_iisy11_r1300/collision/link_4.stl"/>
+        </geometry>
+        <origin rpy="0 0 0" xyz="0 0 0"/>
+      </collision>
+      <inertial>
+        <inertia ixx="0.0283133115058557" ixy="0.0" ixz="0.0" iyy="0.15625788909506" iyz="0.0" izz="0.163792683235523"/>
+        <mass value="7.09182257561761"/>
+        <origin rpy="1.4927296069780172 -1.403978512066052 -1.5036439267584298" xyz="-0.00007163989476214221 0.0445982847464326 -0.175445521620292"/>
+      </inertial>
+      <visual>
+        <geometry>
+          <mesh filename="package://kuka_lbr_iisy_support/meshes/lbr_iisy11_r1300/visual/link_4.stl"/>
+        </geometry>
+        <origin rpy="0 0 0" xyz="0 0 0"/>
+        <xacro:material_kuka_ral_pure_white/>
+      </visual>
+    </link>
+    <link name="${prefix}link_5">
+      <collision>
+        <geometry>
+          <mesh filename="package://kuka_lbr_iisy_support/meshes/lbr_iisy11_r1300/collision/link_5.stl"/>
+        </geometry>
+        <origin rpy="0 0 0" xyz="0 0 0"/>
+      </collision>
+      <inertial>
+        <inertia ixx="0.00667288072123254" ixy="0.0" ixz="0.0" iyy="0.00503543168148481" iyz="0.0" izz="0.00841044585602456"/>
+        <mass value="2.4516241997261"/>
+        <origin rpy="0.4256203528755516 0.14544264795709014 1.2195648324165669" xyz="0.0384076101043046 0.00235993465013012 -0.0244545111288499"/>
+      </inertial>
+      <visual>
+        <geometry>
+          <mesh filename="package://kuka_lbr_iisy_support/meshes/lbr_iisy11_r1300/visual/link_5.stl"/>
+        </geometry>
+        <origin rpy="0 0 0" xyz="0 0 0"/>
+        <xacro:material_kuka_ral_pure_white/>
+      </visual>
+    </link>
+    <link name="${prefix}link_6">
+      <collision>
+        <geometry>
+          <mesh filename="package://kuka_lbr_iisy_support/meshes/lbr_iisy11_r1300/collision/link_6.stl"/>
+        </geometry>
+        <origin rpy="0 0 0" xyz="0 0 0"/>
+      </collision>
+      <inertial>
+        <inertia ixx="0.00390274036654823" ixy="0.0" ixz="0.0" iyy="0.00286930887521153" iyz="0.0" izz="0.00403512413298348"/>
+        <mass value="1.23566751268437"/>
+        <origin rpy="-0.051936335875096745 -0.1296523529795729 -0.0038347791577379832" xyz="0.00315856028595676 0.0135678555121583 -0.038876254431844504"/>
+      </inertial>
+      <visual>
+        <geometry>
+          <mesh filename="package://kuka_lbr_iisy_support/meshes/lbr_iisy11_r1300/visual/link_6.stl"/>
+        </geometry>
+        <origin rpy="0 0 0" xyz="0 0 0"/>
+        <xacro:material_kuka_ral_pure_white/>
+      </visual>
+    </link>
+    <joint name="${prefix}world-waybo_base" type="fixed">
+      <parent link="world"/>
+      <child link="waybo_base"/>
+      <origin rpy="0 0 0" xyz="0 0 0"/>
+    </joint>
+    <joint name="waybo_base-${prefix}base_link" type="fixed">
+      <parent link="waybo_base"/>
+      <child link="${prefix}base_link"/>
+      <origin rpy="-0.4636 0.0 -0.0" xyz="-0.1 0.5 0.76"/>
+    </joint>
+    <joint name="${prefix}joint_1" type="revolute">
+      <axis xyz="0.0 0.0 1.0"/>
+      <child link="${prefix}link_1"/>
+      <limit effort="405.84" lower="-3.2288591125" upper="3.2288591125" velocity="3.49065850398866"/>
+      <origin rpy="${pi} 0 0" xyz="0.0 0.0 0.1845"/>
+      <parent link="${prefix}base_link"/>
+    </joint>
+    <joint name="${prefix}joint_2" type="revolute">
+      <axis xyz="0.0 0.0 1.0"/>
+      <child link="${prefix}link_2"/>
+      <limit effort="366.247685" lower="-4.014257279586958" upper="0.8726646259971648" velocity="3.490656"/>
+      <origin rpy="${pi/2.0} 0 -0" xyz="0.0 0.1011 -0.1155"/>
+      <parent link="${prefix}link_1"/>
+    </joint>
+    <joint name="${prefix}joint_3" type="revolute">
+      <axis xyz="0.0 0.0 1.0"/>
+      <child link="${prefix}link_3"/>
+      <limit effort="147.189439778934" lower="-2.617993875" upper="2.617993875" velocity="3.49065850398866"/>
+      <origin rpy="0 -0 0" xyz="0.59 0 0.0237"/>
+      <parent link="${prefix}link_2"/>
+    </joint>
+    <joint name="${prefix}joint_4" type="revolute">
+      <axis xyz="0.0 0.0 1.0"/>
+      <child link="${prefix}link_4"/>
+      <limit effort="65.4825468125571" lower="-3.14159265" upper="3.14159265" velocity="4.01425727958696"/>
+      <origin rpy="${pi/2} 0 ${-pi/2}" xyz="0.1139 0 0.0774"/>
+      <parent link="${prefix}link_3"/>
+    </joint>
+    <joint name="${prefix}joint_5" type="revolute">
+      <axis xyz="0.0 0.0 1.0"/>
+      <child link="${prefix}link_5"/>
+      <limit effort="64.6576468348751" lower="-1.919862175" upper="1.919862175" velocity="4.53785605518526"/>
+      <origin rpy="0 ${pi/2} ${pi/2}" xyz="0 0.0507 -0.4181"/>
+      <parent link="${prefix}link_4"/>
+    </joint>
+    <joint name="${prefix}joint_6" type="revolute">
+      <axis xyz="0.0 0.0 1.0"/>
+      <child link="${prefix}link_6"/>
+      <limit effort="15.7202326869092" lower="-3.83972435" upper="3.83972435" velocity="7.50491578357562"/>
+      <origin rpy="${pi/2} 0 ${-pi/2}" xyz="0.0837 0 -0.0507"/>
+      <parent link="${prefix}link_5"/>
+    </joint>
+    <!-- ROS-Industrial 'base' frame - equivalent of 'KUKA ROBROOT'-->
+    <link name="${prefix}base"/>
+    <joint name="${prefix}base_link-base" type="fixed">
+      <origin xyz="0 0 0" rpy="0 0 0"/>
+      <parent link="${prefix}base_link"/>
+      <child link="${prefix}base"/>
+    </joint>
+    <!-- ROS-Industrial 'flange' frame - attachment point for EEF models -->
+    <link name="${prefix}flange"/>
+    <joint name="${prefix}link6-flange" type="fixed">
+      <child link="${prefix}flange"/>
+      <origin rpy="0 ${pi/2} 0" xyz="0 0 -0.0943"/>
+      <parent link="${prefix}link_6"/>
+    </joint>
+    <!-- ROS-Industrial 'tool0' frame - all-zeros tool frame -->
+    <link name="${prefix}tool0"/>
+    <joint name="${prefix}link6-tool0" type="fixed">
+      <child link="${prefix}tool0"/>
+      <origin rpy="0 ${pi} 0" xyz="0 0 -0.0943"/>
+      <parent link="${prefix}link_6"/>
+    </joint>
+  </xacro:macro>
+  <xacro:kuka_lbr_iisy11_r1300_robot prefix="$(arg prefix)" controller_ip="$(arg controller_ip)" client_ip="$(arg client_ip)" use_fake_hardware="$(arg use_fake_hardware)" roundtrip_time="$(arg roundtrip_time)" qos_config_file="$(arg qos_config_file)">
+    <origin xyz="$(arg x) $(arg y) $(arg z)" rpy="$(arg roll) $(arg pitch) $(arg yaw)"/>
+  </xacro:kuka_lbr_iisy11_r1300_robot>
+</robot>
+<!-- <?xml version="1.0"?>
+<robot xmlns:xacro="http://www.ros.org/wiki/xacro" name="lbr_iisy11_r1300">
   <xacro:include filename="$(find kuka_lbr_iisy_support)/urdf/lbr_iisy11_r1300_macro.xacro"/>
-  <!-- Read additional arguments  -->
   <xacro:arg name="prefix" default=""/>
   <xacro:arg name="controller_ip" default="0.0.0.0"/>
@@ -19,3 +266,52 @@
     <origin xyz="$(arg x) $(arg y) $(arg z)" rpy="$(arg roll) $(arg pitch) $(arg yaw)"/>
   </xacro:kuka_lbr_iisy11_r1300_robot>
-</robot>
+</robot> -->
+<!-- <?xml version="1.0"?>
+<robot xmlns:xacro="http://www.ros.org/wiki/xacro" name="lbr_iisy11_r1300">
+  <xacro:include filename="$(find kuka_lbr_iisy_support)/urdf/lbr_iisy11_r1300_macro.xacro"/>
+  Read additional arguments
+  <xacro:arg name="prefix" default=""/>
+  <xacro:arg name="controller_ip" default="0.0.0.0"/>
+  <xacro:arg name="client_ip" default="0.0.0.0"/>
+  <xacro:arg name="use_fake_hardware" default="false"/>
+  <xacro:arg name="roundtrip_time" default="0"/>
+  <xacro:arg name="qos_config_file" default=""/>
+  <xacro:arg name="x" default="0"/>
+  <xacro:arg name="y" default="0"/>
+  <xacro:arg name="z" default="0"/>
+  <xacro:arg name="roll" default="0"/>
+  <xacro:arg name="pitch" default="0"/>
+  <xacro:arg name="yaw" default="0"/>
+  <link name="waybo_base">
+    <inertial>
+      <origin xyz="0.0 0.0 0.0" rpy="0 0 0"/>
+      <mass value="50.0"/>
+      <inertia ixx="10.0" ixy="0.0" ixz="0.0" iyy="10.0" iyz="0.0" izz="10.0"/>
+    </inertial>
+    <visual>
+      <origin xyz="0.0 0.0 0.0" rpy="0 0 0"/>
+      <geometry>
+        <mesh filename="package://kuka_lbr_iisy_support/meshes/waybo_base.STL"/>
+      </geometry>
+    </visual>
+    <collision>
+      <origin xyz="0.0 0.0 0.0" rpy="0 0 0"/>
+      <geometry>
+        <mesh filename="package://kuka_lbr_iisy_support/meshes/waybo_base.STL"/>
+      </geometry>
+    </collision>
+  </link>
+  <joint name="world_to_waybo_base" type="fixed">
+    <parent link="world"/>
+    <child link="waybo_base"/>
+    <origin xyz="0.0 0.0 0.98" rpy="-0.3828 -0.3828 -0.3962"/>
+  </joint>
+  <joint name="waybo_base_to_base_link" type="fixed">
+    <parent link="waybo_base"/>
+    <child link="${prefix}base_link"/>
+    <origin xyz="0.0 0.0 0.0" rpy="0 0 0"/>
+  </joint>
+  <xacro:kuka_lbr_iisy11_r1300_robot prefix="$(arg prefix)" controller_ip="$(arg controller_ip)" client_ip="$(arg client_ip)" use_fake_hardware="$(arg use_fake_hardware)" roundtrip_time="$(arg roundtrip_time)" qos_config_file="$(arg qos_config_file)">
+    <origin xyz="$(arg x) $(arg y) $(arg z)" rpy="$(arg roll) $(arg pitch) $(arg yaw)"/>
+  </xacro:kuka_lbr_iisy11_r1300_robot>
+</robot> -->
