Commit message: waybo_base with lbr_iisy11

File: kuka_lbr_iisy_support/urdf/lbr_iisy11_r1300_macro.xacro (robot description, xacro)
@@ -15,5 +15,5 @@
           <mesh filename="package://kuka_lbr_iisy_support/meshes/lbr_iisy11_r1300/collision/base_link.stl"/>
         </geometry>
-        <origin rpy="-0.0 0.0 -0.0" xyz="0.0 0.0 0.0"/>
+        <origin rpy="0 0 0" xyz="0.0 0.0 0.0"/>
       </collision>
       <visual>
@@ -21,5 +21,5 @@
           <mesh filename="package://kuka_lbr_iisy_support/meshes/lbr_iisy11_r1300/visual/base_link.stl"/>
         </geometry>
-        <origin rpy="-0.0 0.0 -0.0" xyz="0.0 0.0 0.0"/>
+        <origin rpy="0 0 0" xyz="0.0 0.0 0.0"/>
         <xacro:material_kuka_ral_pure_white/>
       </visual>
@@ -30,10 +30,10 @@
           <mesh filename="package://kuka_lbr_iisy_support/meshes/lbr_iisy11_r1300/collision/link_1.stl"/>
         </geometry>
-        <origin rpy="-0.0 0.0 -0.0" xyz="0.0 0.0 0.0"/>
+        <origin rpy="0 0 0" xyz="0.0 0.0 0.0"/>
       </collision>
       <inertial>
         <inertia ixx="0.0489108039022503" ixy="0.0" ixz="0.0" iyy="0.038370593540088" iyz="0.0" izz="0.0522121642769911"/>
         <mass value="9.62E0"/>
-        <origin rpy="-1.3035636348359196 -0.7815781053554712 1.2529437882898178" xyz="0.00344301039501039 0.0191980353430353 -0.08662803846153849"/>
+        <origin rpy="0 0 0" xyz="0.00344301039501039 0.0191980353430353 -0.08662803846153849"/>
       </inertial>
       <visual>
@@ -41,5 +41,5 @@
           <mesh filename="package://kuka_lbr_iisy_support/meshes/lbr_iisy11_r1300/visual/link_1.stl"/>
         </geometry>
-        <origin rpy="-0.0 0.0 -0.0" xyz="0.0 0.0 0.0"/>
+        <origin rpy="0 0 0" xyz="0.0 0.0 0.0"/>
         <xacro:material_kuka_ral_pure_white/>
       </visual>
@@ -50,10 +50,10 @@
           <mesh filename="package://kuka_lbr_iisy_support/meshes/lbr_iisy11_r1300/collision/link_2.stl"/>
         </geometry>
-        <origin rpy="-0.0 0.0 -0.0" xyz="0.0 0.0 0.0"/>
+        <origin rpy="0 0 0" xyz="0.0 0.0 0.0"/>
       </collision>
       <inertial>
         <inertia ixx="0.609923712050298" ixy="0.0" ixz="0.0" iyy="0.0385097671170806" iyz="0.0" izz="0.617803845441985"/>
         <mass value="9.86515786038357E0"/>
-        <origin rpy="-0.0037282594736534596 -0.018939981545576166 -1.569953728930981" xyz="0.249085185084359 -0.00442629366790902 -0.0535128397562821"/>
+        <origin rpy="0 0 0" xyz="0.249085185084359 -0.00442629366790902 -0.0535128397562821"/>
       </inertial>
       <visual>
@@ -61,5 +61,5 @@
           <mesh filename="package://kuka_lbr_iisy_support/meshes/lbr_iisy11_r1300/visual/link_2.stl"/>
         </geometry>
-        <origin rpy="-0.0 0.0 -0.0" xyz="0.0 0.0 0.0"/>
+        <origin rpy="0 0 0" xyz="0.0 0.0 0.0"/>
         <xacro:material_kuka_ral_pure_white/>
       </visual>
@@ -70,5 +70,5 @@
           <mesh filename="package://kuka_lbr_iisy_support/meshes/lbr_iisy11_r1300/collision/link_3.stl"/>
         </geometry>
-        <origin rpy="-0.0 0.0 -0.0" xyz="0.0 0.0 0.0"/>
+        <origin rpy="0 0 0" xyz="0.0 0.0 0.0"/>
       </collision>
       <inertial>
@@ -81,5 +81,5 @@
           <mesh filename="package://kuka_lbr_iisy_support/meshes/lbr_iisy11_r1300/visual/link_3.stl"/>
         </geometry>
-        <origin rpy="-0.0 0.0 -0.0" xyz="0.0 0.0 0.0"/>
+        <origin rpy="0 0 0" xyz="0.0 0.0 0.0"/>
         <xacro:material_kuka_ral_pure_white/>
       </visual>
@@ -90,10 +90,10 @@
           <mesh filename="package://kuka_lbr_iisy_support/meshes/lbr_iisy11_r1300/collision/link_4.stl"/>
         </geometry>
-        <origin rpy="-0.0 0.0 -0.0" xyz="0.0 0.0 0.0"/>
+        <origin rpy="0 0 0" xyz="0.0 0.0 0.0"/>
       </collision>
       <inertial>
         <inertia ixx="0.0283133115058557" ixy="0.0" ixz="0.0" iyy="0.15625788909506" iyz="0.0" izz="0.163792683235523"/>
         <mass value="7.09182257561761E0"/>
-        <origin rpy="1.4927296069780172 -1.403978512066052 -1.5036439267584298" xyz="-7.163989476214221E-5 0.0445982847464326 -0.175445521620292"/>
+        <origin rpy="0 0 0" xyz="-7.163989476214221E-5 0.0445982847464326 -0.175445521620292"/>
       </inertial>
       <visual>
@@ -101,5 +101,5 @@
           <mesh filename="package://kuka_lbr_iisy_support/meshes/lbr_iisy11_r1300/visual/link_4.stl"/>
         </geometry>
-        <origin rpy="-0.0 0.0 -0.0" xyz="0.0 0.0 0.0"/>
+        <origin rpy="0 0 0" xyz="0.0 0.0 0.0"/>
         <xacro:material_kuka_ral_pure_white/>
       </visual>
@@ -110,5 +110,5 @@
           <mesh filename="package://kuka_lbr_iisy_support/meshes/lbr_iisy11_r1300/collision/link_5.stl"/>
         </geometry>
-        <origin rpy="-0.0 0.0 -0.0" xyz="0.0 0.0 0.0"/>
+        <origin rpy="0 0 0" xyz="0.0 0.0 0.0"/>
       </collision>
       <inertial>
@@ -121,5 +121,5 @@
           <mesh filename="package://kuka_lbr_iisy_support/meshes/lbr_iisy11_r1300/visual/link_5.stl"/>
         </geometry>
-        <origin rpy="-0.0 0.0 -0.0" xyz="0.0 0.0 0.0"/>
+        <origin rpy="0 0 0" xyz="0.0 0.0 0.0"/>
         <xacro:material_kuka_ral_pure_white/>
       </visual>
@@ -130,10 +130,10 @@
           <mesh filename="package://kuka_lbr_iisy_support/meshes/lbr_iisy11_r1300/collision/link_6.stl"/>
         </geometry>
-        <origin rpy="-0.0 0.0 -0.0" xyz="0.0 0.0 0.0"/>
+        <origin rpy="0 0 0" xyz="0.0 0.0 0.0"/>
       </collision>
       <inertial>
         <inertia ixx="0.00390274036654823" ixy="0.0" ixz="0.0" iyy="0.00286930887521153" iyz="0.0" izz="0.00403512413298348"/>
         <mass value="1.23566751268437E0"/>
-        <origin rpy="-0.051936335875096745 -0.1296523529795729 -0.0038347791577379832" xyz="0.00315856028595676 0.0135678555121583 -0.038876254431844504"/>
+        <origin rpy="0 0 0" xyz="0.00315856028595676 0.0135678555121583 -0.038876254431844504"/>
       </inertial>
       <visual>
@@ -141,5 +141,5 @@
           <mesh filename="package://kuka_lbr_iisy_support/meshes/lbr_iisy11_r1300/visual/link_6.stl"/>
         </geometry>
-        <origin rpy="-0.0 0.0 -0.0" xyz="0.0 0.0 0.0"/>
+        <origin rpy="0 0 0" xyz="0.0 0.0 0.0"/>
         <xacro:material_kuka_ral_pure_white/>
       </visual>
@@ -149,5 +149,5 @@
       <parent link="world"/>
       <child link="${prefix}base_link"/>
-      <xacro:insert_block name="origin"/>
+      <origin rpy="0 -0.3828 0" xyz="0.0 0.0 1.002"/>
     </joint>
     <joint name="${prefix}joint_1" type="revolute">
@@ -155,5 +155,5 @@
       <child link="${prefix}link_1"/>
       <limit effort="4.0584E2" lower="-3.2288591125E0" upper="3.2288591125E0" velocity="3.49065850398866E0"/>
-      <origin rpy="${pi} -0.0 0.0" xyz="0.0 0.0 0.1845"/>
+      <origin rpy="${pi} 0 0" xyz="0.0 0.0 0.1845"/>
       <parent link="${prefix}base_link"/>
     </joint>
@@ -162,5 +162,5 @@
       <child link="${prefix}link_2"/>
       <limit effort="366.247685" lower="-4.014257279586958E0" upper="8.726646259971648E-1" velocity="3.490656"/>
-      <origin rpy="${pi/2.0} 0.0 -0.0" xyz="0.0 0.1011 -0.1155"/>
+      <origin rpy="${pi/2.0} 0 0" xyz="0.0 0.1011 -0.1155"/>
       <parent link="${prefix}link_1"/>
     </joint>
@@ -169,5 +169,5 @@
       <child link="${prefix}link_3"/>
       <limit effort="1.47189439778934E2" lower="-2.617993875E0" upper="2.617993875E0" velocity="3.49065850398866E0"/>
-      <origin rpy="0.0 -0.0 0.0" xyz="0.59 0.0 0.0237"/>
+      <origin rpy="0 0 0" xyz="0.59 0.0 0.0237"/>
       <parent link="${prefix}link_2"/>
     </joint>
@@ -176,5 +176,5 @@
       <child link="${prefix}link_4"/>
       <limit effort="6.54825468125571E1" lower="-3.14159265E0" upper="3.14159265E0" velocity="4.01425727958696E0"/>
-      <origin rpy="${pi/2} -0.0 ${-pi/2}" xyz="0.1139 0.0 0.0774"/>
+      <origin rpy="${pi/2} 0 ${-pi/2}" xyz="0.1139 0.0 0.0774"/>
       <parent link="${prefix}link_3"/>
     </joint>
@@ -183,5 +183,5 @@
       <child link="${prefix}link_5"/>
       <limit effort="6.46576468348751E1" lower="-1.919862175E0" upper="1.919862175E0" velocity="4.53785605518526E0"/>
-      <origin rpy="0.0 ${pi/2} ${pi/2}" xyz="0.0 0.0507 -0.4181"/>
+      <origin rpy="0 ${pi/2} ${pi/2}" xyz="0.0 0.0507 -0.4181"/>
       <parent link="${prefix}link_4"/>
     </joint>
@@ -190,5 +190,5 @@
       <child link="${prefix}link_6"/>
       <limit effort="1.57202326869092E1" lower="-3.83972435E0" upper="3.83972435E0" velocity="7.50491578357562E0"/>
-      <origin rpy="${pi/2} -0.0 ${-pi/2}" xyz="0.0837 0.0 -0.0507"/>
+      <origin rpy="${pi/2} 0 ${-pi/2}" xyz="0.0837 0.0 -0.0507"/>
       <parent link="${prefix}link_5"/>
     </joint>
@@ -204,5 +204,5 @@
     <joint name="${prefix}link6-flange" type="fixed">
       <child link="${prefix}flange"/>
-      <origin rpy="0.0 ${pi/2} 0.0" xyz="0.0 0.0 -0.0943"/>
+      <origin rpy="0 ${pi/2} 0" xyz="0.0 0.0 -0.0943"/>
       <parent link="${prefix}link_6"/>
     </joint>
@@ -211,7 +211,14 @@
     <joint name="${prefix}link6-tool0" type="fixed">
       <child link="${prefix}tool0"/>
-      <origin rpy="0.0 ${pi} 0.0" xyz="0.0 0.0 -0.0943"/>
+      <origin rpy="0 ${pi} 0" xyz="0.0 0.0 -0.0943"/>
       <parent link="${prefix}link_6"/>
     </joint>
   </xacro:macro>
+  <!-- Include the Waybo base -->
+  <xacro:include filename="$(find kuka_lbr_iisy_support)/urdf/waybo.urdf"/>
+  <joint name="waybo_base_to_base_link" type="fixed">
+    <parent link="${prefix}waybo_base_link"/>
+    <child link="${prefix}base_link"/>
+    <origin rpy="0 0 0" xyz="0 0 1.0"/>
+  </joint>
 </robot>

Commit message: fixed base_pose for robot

File: kuka_lbr_iisy_support/urdf/lbr_iisy11_r1300.urdf.xacro (robot description, xacro)
@@ -178,5 +178,5 @@
       <parent link="waybo_base"/>
       <child link="${prefix}base_link"/>
-      <origin rpy="-0.4636 0.0 -0.0" xyz="-0.1 0.5 0.76"/>
+      <origin rpy="-0.387 -0.361 -0.857" xyz="-0.1 0.5 0.76"/>
     </joint>
     <joint name="${prefix}joint_1" type="revolute">
